File: PrismDDIN18.sch (KiCad schematic (older format))
At the start: 85 parts, among them CON1 BARREL_JACK, IC1 LM2596T-5, IC2 MEGA8-P, M1 IN-18, M10 IN-18, P1 ESP8266-01_02X04, Q1 16MHz, Q2 BSS138, Q3 BSS138, Q4 IRF540N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

Commit message: Update to KiCAD 5, re-space
Parts:
- 2N3906: symbol Q_PNP_BCE -> PrismDDIN18-rescue:Q_PNP_BCE
- C1, C13, C14, C2, C3, C4, C5, C6: symbol C_Small -> PrismDDIN18-rescue:C_Small
- C10, C11, C7, C8, C9: symbol RCL_C-EU050-024X044 -> PrismDDIN18-rescue:RCL_C-EU050-024X044
- C12, C15, C16, C17, C20: symbol CP -> PrismDDIN18-rescue:CP
- C18, C19: symbol C -> PrismDDIN18-rescue:C
- CON1: symbol BARREL_JACK -> PrismDDIN18-rescue:BARREL_JACK
- D1, D2, D3, D4: symbol D-RESCUE-KickstarterNixie -> PrismDDIN18-rescue:D-RESCUE-KickstarterNixie
- D5, D6, D7, D8: symbol LED -> PrismDDIN18-rescue:LED
- H1, H10, M1, M10, S1, S10: symbol IN-18 -> PrismDDIN18-rescue:IN-18
- IC1: symbol LM2596T-5 -> PrismDDIN18-rescue:LM2596T-5
- IC2: symbol ATMEL_MEGA8-P -> PrismDDIN18-rescue:ATMEL_MEGA8-P
- L1: symbol RCL_L-US6000-XXX-RC -> PrismDDIN18-rescue:RCL_L-US6000-XXX-RC
- L2: value 33uH -> 100uH; symbol RCL_L-US6000-XXX-RC -> PrismDDIN18-rescue:RCL_L-US6000-XXX-RC
- LED1, LED2, LED3, LED4, LED5, LED6: symbol WS2812B -> PrismDDIN18-rescue:WS2812B
- LED7: symbol LED_LED3MM -> PrismDDIN18-rescue:LED_LED3MM
- P1: symbol ESP8266-01_02X04 -> PrismDDIN18-rescue:ESP8266-01_02X04
- Q1: symbol CRYSTAL_CRYSTALHC49S -> PrismDDIN18-rescue:CRYSTAL_CRYSTALHC49S
- Q2, Q3: symbol Q_NMOS_GSD -> PrismDDIN18-rescue:Q_NMOS_GSD
- Q4: symbol IRF540N-RESCUE-DDIN18 -> PrismDDIN18-rescue:IRF540N-RESCUE-DDIN18
- R1, R10, R11, R12, R13, R15, R16, R17, R18, R19, R2, R20, R21, R3, R4, R5, R6: symbol R -> PrismDDIN18-rescue:R
- R14: value R -> 0R22 2W; symbol R -> PrismDDIN18-rescue:R
- R7, R8, R9: symbol RCL_R-EU_0207/2V -> PrismDDIN18-rescue:RCL_R-EU_0207_2V
- RV1: symbol POT -> PrismDDIN18-rescue:POT
- SV1, SV4: symbol CONN_01X04 -> PrismDDIN18-rescue:CONN_01X04
- SV2: symbol CONN_01X05 -> PrismDDIN18-rescue:CONN_01X05
- SV3: symbol CON-LSTB_MA03-2 -> PrismDDIN18-rescue:CON-LSTB_MA03-2
- U1: symbol AP111733 -> PrismDDIN18-rescue:AP111733
- U2: symbol MC34063A -> PrismDDIN18-rescue:MC34063A
- U3, U4: symbol HV5622 -> PrismDDIN18-rescue:HV5622
- W1, W2, W3: symbol TEST_1P -> PrismDDIN18-rescue:TEST_1P
Connections:
- wire segments 426 -> 516
Other:
- note added: "Display drivers"
- note added: "NeoPixel back lights"
- note added: "Tubes"
- moved on the sheet: C1, C2, C3, C4, C5, C6, CON1, D5, D6, D7, D8, H1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

Commit message: Added DS1307, re-laid out HV
Parts:
- added BT1: Battery_Cell, NixieClockMaster:CR1220-CoinCell, symbol Device:Battery_Cell
- added C21: C, NixieClockMaster:C025-024X044, symbol Device:C
- added U5: DS1307+, Package_DIP:DIP-8_W7.62mm, symbol Timer_RTC:DS1307+
- added Y1: Crystal_Small, NixieClockMaster:Crystal_DS10_d1.0mm_l4.3mm_Horizontal, symbol Device:Crystal_Small
- U1: value AP111733 -> AMS1117-3V3; symbol PrismDDIN18-rescue:AP111733 -> Regulator_Linear:AMS1117-3.3
Connections:
- net GND: now also BT1.2 (-), C21.2, U5.4 (GND)
- net SCL: now also U5.6 (SCL)
- net SDA: now also U5.5 (SDA)
- net VCC: now also C21.1, U5.8 (VCC)
- new net: U5.1 (X1), Y1.1
- new net: U5.2 (X2), Y1.2
- new net: BT1.1 (+), U5.3 (VBAT)
- no-connect marks 17 -> 18
Other:
- note added: "Barrel Jack Input"
- note added: "Front panel"
- note added: "I2C interface"
- note added: "ICSP programming port"
- note removed: "Connections"
- moved on the sheet: CON1, R9, SV2, SV4, U1, W2
