File: PrismDDIN18.kicad_pcb (KiCad board)
At the start: 2 copper layers, 229.9 x 54.6 mm, 85 parts, among them CON1 BARREL_JACK, IC1 LM2596T-5, IC2 MEGA8-P, M1 IN-18, M10 IN-18, P1 ESP8266-01_02X04, Q1 16MHz, Q2 BSS138, Q3 BSS138, Q4 IRF540N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

Commit message: Update to KiCAD 5, re-space
Parts:
- moved Q3 101.3 mm to (341.9, 142.9)
- moved R12 101.3 mm to (336.1, 152.1)
- moved C6 101.3 mm to (339.9, 130.0)
- moved H10 101.3 mm to (340.0, 125.0)
- moved LED6 101.3 mm to (339.8, 124.9)
- moved LED7 101.3 mm to (353.7, 139.6)
- moved P1 101.3 mm to (349.0, 154.4)
- moved Q2 101.3 mm to (341.9, 146.5)
- moved R1 101.3 mm to (336.3, 110.3)
- moved R10 101.3 mm to (334.8, 146.5)
- moved R11 101.3 mm to (334.7, 142.9)
- moved R13 101.3 mm to (339.1, 152.1)
- moved SV4 101.3 mm to (356.5, 150.3)
- moved C13 101.3 mm to (333.2, 152.1)
- moved C14 101.3 mm to (342.0, 152.1)
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Routing:
- net /VCC: track 548.9 -> 620.5 mm
- net /HV: track 272.5 -> 326.5 mm
- net /PWR_VIN: track 212.2 -> 253.4 mm
- net /DATA0: track 146.9 -> 175.5 mm
- net /BLANK: track 146.3 -> 173.1 mm
- net /H1_7: track 42.2 -> 67.9 mm, vias 1 -> 2
- net /H1_6: track 49.2 -> 72.7 mm, vias 0 -> 1
- net /CLK: track 103.1 -> 125.6 mm
- net /LATCH: track 115.2 -> 137.5 mm
- net /SCL: track 160.2 -> 181.0 mm
- net /SDA: track 167.3 -> 187.9 mm
- net /M1_4: track 45.3 -> 64.8 mm
- net /M1_3: track 26.1 -> 45.5 mm
- net /M1_8: track 25.1 -> 44.4 mm
- net /M1_2: track 16.9 -> 36.2 mm
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Other:
- board size 229.9 x 54.6 mm -> 280 x 70 mm

Commit message: Shrink board to 280x60
Other:
- board size 280 x 70 mm -> 280 x 60 mm
Changed lines of the file:
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@@
       (net 17 /PWR_VIN))
   )
-  (gr_line (start 80 170) (end 80 100) (angle 90) (layer Edge.Cuts) (width 0.15))
-  (gr_line (start 360 170) (end 80 170) (angle 90) (layer Edge.Cuts) (width 0.15))
-  (gr_line (start 360 100) (end 360 170) (angle 90) (layer Edge.Cuts) (width 0.15))
-  (gr_line (start 80 100) (end 360 100) (angle 90) (layer Edge.Cuts) (width 0.15))
+  (gr_line (start 80 166) (end 80 106) (angle 90) (layer Edge.Cuts) (width 0.15))
+  (gr_line (start 360 166) (end 80 166) (angle 90) (layer Edge.Cuts) (width 0.15))
+  (gr_line (start 360 106) (end 360 166) (angle 90) (layer Edge.Cuts) (width 0.15))
+  (gr_line (start 80 106) (end 360 106) (angle 90) (layer Edge.Cuts) (width 0.15))
   (segment (start 303.9243 111.4418) (end 302.0828 111.4418) (width 0.25) (layer F.Cu) (net 1) (status 10))
   (segment (start 302.0828 111.4418) (end 300 113.5246) (width 0.25) (layer F.Cu) (net 1))
@@
   (segment (start 311.791111 119.156211) (end 311.791111 133.877189) (width 0.25) (layer B.Cu) (net 47))
   (via (at 264.96 116.78) (size 0.6) (drill 0.4) (layers F.Cu B.Cu) (net 48))
-  (segment (start 264.96 131.09) (end 264.96 116.78) (width 0.25) (layer B.Cu) (net 48))
-  (segment (start 266.61 132.74) (end 264.96 131.09) (width 0.25) (layer B.Cu) (net 48))
-  (segment (start 264.14 151.95) (end 264.14 147.494998) (width 0.25) (layer B.Cu) (net 48))
-  (segment (start 265.35 153.16) (end 264.14 151.95) (width 0.25) (layer B.Cu) (net 48))
-  (segment (start 267.55 144.084998) (end 267.55 139.95) (width 0.25) (layer B.Cu) (net 48))
-  (segment (start 264.14 147.494998) (end 267.55 144.084998) (width 0.25) (layer B.Cu) (net 48))
-  (segment (start 266.61 139.01) (end 266.61 132.74) (width 0.25) (layer B.Cu) (net 48))
-  (segment (start 267.55 139.95) (end 266.61 139.01) (width 0.25) (layer B.Cu) (net 48))
   (segment (start 267.330011 114.409989) (end 265.259999 116.480001) (width 0.25) (layer F.Cu) (net 48))
   (segment (start 265.259999 116.480001) (end 264.96 116.78) (width 0.25) (layer F.Cu) (net 48))
   (segment (start 293.930869 114.409989) (end 267.330011 114.409989) (width 0.25) (layer F.Cu) (net 48))
   (segment (start 296.30176 116.78088) (end 293.930869 114.409989) (width 0.25) (layer F.Cu) (net 48))
+  (segment (start 266.61 139.01) (end 266.61 132.74) (width 0.25) (layer B.Cu) (net 48))
+  (segment (start 264.14 147.494998) (end 267.55 144.084998) (width 0.25) (layer B.Cu) (net 48))
+  (segment (start 267.55 139.95) (end 266.61 139.01) (width 0.25) (layer B.Cu) (net 48))
+  (segment (start 267.55 144.084998) (end 267.55 139.95) (width 0.25) (layer B.Cu) (net 48))
+  (segment (start 265.35 153.16) (end 264.14 151.95) (width 0.25) (layer B.Cu) (net 48))
+  (segment (start 264.14 151.95) (end 264.14 147.494998) (width 0.25) (layer B.Cu) (net 48))
+  (segment (start 266.61 132.74) (end 264.96 131.09) (width 0.25) (layer B.Cu) (net 48))
+  (segment (start 264.96 131.09) (end 264.96 116.78) (width 0.25) (layer B.Cu) (net 48))
   (segment (start 262.81 150.62) (end 262.81 149.6715) (width 0.25) (layer F.Cu) (net 49))
   (segment (start 262.81 149.6715) (end 265.3115 147.17) (width 0.25) (layer F.Cu) (net 49))
@@
     (polygon
       (pts
-        (xy 80 100.01) (xy 80.01 170) (xy 360 169.99) (xy 360 100)
+        (xy 80.01 106.01) (xy 80.01 166) (xy 360 166) (xy 360 106)
       )
     )

Commit message: Added DS1307, re-laid out HV
Parts:
- added BT1: Battery_Cell, NixieClockMaster:CR1220-CoinCell, F.Cu at (180.9, 153.8)
- added C21: C, NixieClockMaster:C025-024X044, F.Cu at (282.7, 150.4)
- added MH1: MountingHole_3.2mm_M3, NixieClockMaster:MountingHole_3.2mm_M3, F.Cu at (356.5, 162.5)
- added MH1: MountingHole_3.2mm_M3, NixieClockMaster:MountingHole_3.2mm_M3, F.Cu at (356.4, 109.6)
- added MH1: MountingHole_3.2mm_M3, NixieClockMaster:MountingHole_3.2mm_M3, F.Cu at (83.6, 109.7)
- added MH1: MountingHole_3.2mm_M3, NixieClockMaster:MountingHole_3.2mm_M3, F.Cu at (83.6, 162.2)
- added U5: DS1307+, Package_DIP:DIP-8_W7.62mm, F.Cu at (285.6, 154.1)
- added Y1: Crystal_Small, NixieClockMaster:Crystal_DS10_d1.0mm_l4.3mm_Horizontal, F.Cu at (286.0, 156.5)
- 2N3906: footprint NixieClockMaster:2N7000_TO92 -> NixieClockMaster:TO-92_inline
- C20: footprint NixieClockMaster:C_Radial_D6.3_L11.2_P2.5 -> NixieClockMaster:C_Radial_D10_L11.2_P2.5_3.5_5
- D1: footprint NixieClockMaster:Diode_DO-41_SOD81_Vertical_AnodeUp -> NixieClockMaster:Diode_DO-41_1N4001
- D3: footprint NixieClockMaster:Diode_DO-41_1N4001 -> NixieClockMaster:Diode_DO-41_SOD81_Vertical_AnodeUp
- L2: value 33uH -> 100uH; footprint NixieClockMaster:Inductor-33mH-TH-SMD -> NixieClockMaster:Inductor-100mH
- Q4: footprint TO_SOT_Packages_THT:TO-220_Neutral123_Horizontal_LargePads -> NixieClockMaster:TO-220-3_H
- R14: value R -> 0R22 2W; footprint NixieClockMaster:R-0207_2V -> NixieClockMaster:R_2W
- U2: footprint Housings_DIP:DIP-8_W7.62mm_LongPads -> Package_DIP:DIP-8_W7.62mm
- moved R15 57.7 mm to (157.7, 160.3), turned to 270 degrees
- moved D3 47.4 mm to (154.7, 162.8), turned to 90 degrees
- moved D4 43.8 mm to (131.3, 164.1), turned to 0 degrees
- moved R9 34.4 mm to (201.9, 158.8), turned to 0 degrees
- moved 2N3906 33.4 mm to (149.5, 159.8), turned to 270 degrees
- moved C17 30.0 mm to (108.5, 161.0), turned to 0 degrees
- moved C16 26.7 mm to (319.2, 161.6), turned to 0 degrees
- moved SV1 21.0 mm to (83.1, 148.6)
- moved R14 20.3 mm to (122.4, 146.1), turned to 270 degrees
- moved R16 17.6 mm to (127.3, 164.1), turned to 180 degrees
- moved CON1 13.7 mm to (100.1, 158.5)
- moved RV1 12.7 mm to (116.6, 163.3)
- moved D1 10.9 mm to (104.6, 148.6)
- moved R17 10.8 mm to (122.2, 164.1), turned to 180 degrees
- moved U2 10.3 mm to (109.2, 151.9)
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Connections:
- R18 pad 1: /HV -> Net-(D6-Pad2)
- R18 pad 2: Net-(D6-Pad2) -> /HV
- R19 pad 1: /HV -> Net-(D5-Pad2)
- R19 pad 2: Net-(D5-Pad2) -> /HV
Routing:
- net GND: track 545.7 -> 174.7 mm, vias 3 -> 4
- net Net-(BT1-Pad1): track 0.00 -> 116.8 mm, vias 0 -> 3
- net Net-(2N3906-Pad1): track 20.5 -> 59.0 mm
- net Net-(C17-Pad1): track 71.7 -> 42.2 mm
- net /SDA: track 187.9 -> 215.6 mm, vias 0 -> 1
- net /SCL: track 181.0 -> 207.1 mm
- net /DLS: track 63.9 -> 38.0 mm
- net Net-(D4-Pad2): track 37.9 -> 21.7 mm
- net /VCC: track 620.5 -> 635.5 mm, vias 13 -> 14
- net Net-(2N3906-Pad3): track 34.3 -> 21.2 mm
- net /HV: track 326.5 -> 338.8 mm, vias 0 -> 2
- net /PWR_INPUT: track 29.0 -> 19.9 mm
- net Net-(D8-Pad1): track 36.3 -> 28.0 mm
- net /PIR: track 28.7 -> 35.2 mm
- net /BTN1: track 30.0 -> 36.6 mm
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
Commit message: Align tubes, add mounting holes
Parts:
- moved R9 23.8 mm to (217.2, 140.5)
- moved R2 6.80 mm to (310.7, 110.3)
- moved R1 6.34 mm to (330.0, 110.3)
- moved R8 5.20 mm to (353.7, 137.3), turned to 180 degrees
- moved LED3 2.22 mm to (200.0, 123.0)
- moved LED4 2.15 mm to (240.0, 123.0)
- moved LED5 2.05 mm to (300.0, 123.0)
- moved H1 1.98 mm to (300.0, 123.0)
- moved H10 1.98 mm to (340.0, 123.0)
- moved M1 1.98 mm to (200.0, 123.0)
- moved M10 1.98 mm to (240.0, 123.0)
- moved C6 1.96 mm to (340.0, 128.0)
- moved LED6 1.93 mm to (340.0, 123.0)
- moved C5 1.81 mm to (300.0, 128.0)
- moved C4 1.63 mm to (240.0, 128.0)
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Routing:
- net /VCC: track 635.5 -> 674.0 mm
- net GND: track 174.7 -> 147.8 mm, vias 4 -> 5
- net /S10_4: track 51.1 -> 59.4 mm, vias 0 -> 1
- net /HV: track 338.8 -> 332.4 mm
- net Net-(H1-PadA): track 7.24 -> 11.7 mm
- net /M1_7: track 55.3 -> 51.3 mm
- net Net-(H10-PadA): track 7.24 -> 11.0 mm
- net /S10_9: track 29.1 -> 32.7 mm, vias 0 -> 1
- net Net-(LED5-Pad4): track 39.9 -> 36.4 mm
- net /DLS: track 38.0 -> 41.2 mm
- net /M1_6: track 60.3 -> 57.3 mm
- net /M1_3: track 45.6 -> 42.6 mm
- net Net-(LED3-Pad4): track 42.9 -> 40.1 mm
- net /M1_4: track 64.6 -> 67.4 mm
- net /H1_4: track 69.1 -> 71.8 mm
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Other:
- board size 280 x 60 mm -> 280 x 62 mm

Commit message: Initial Wemos version
Parts:
- removed C10, C9: 100nF, NixieClockMaster:C025-024X044
- removed C13, C14: 100nF, NixieClockMaster:C_1206_HandSoldering
- removed C15: 10uF, NixieClockMaster:C_1206_HandSoldering
- removed IC2: MEGA8-P, NixieClockMaster:328P_DIL28
- removed P1: ESP8266-01_02X04, NixieClockMaster:ESP8266_2x04
- removed Q1: 16MHz, NixieClockMaster:Crystal_HC49-U_Vertical
- removed SV3: CONN_ISCP, NixieClockMaster:Header_MA03-2
- added J1: Conn_01x03, NixieClockMaster:Header_MA03-1_Small, F.Cu at (357.7, 125.6)
- added Q4: 2N7000, Package_TO_SOT_THT:TO-92_Inline, F.Cu at (191.5, 161.1)
- added Q5: 2N7000, Package_TO_SOT_THT:TO-92_Inline, F.Cu at (191.4, 153.2)
- added R22: 10k, NixieClockMaster:R-0207_2V, F.Cu at (192.7, 150.0)
- added R23: 10k, NixieClockMaster:R-0207_2V, F.Cu at (187.7, 158.0)
- added R24: 10k, NixieClockMaster:R-0207_2V, F.Cu at (187.6, 150.1)
- C7: value 22pF -> 100nF
- C8: value 22pF -> 220uF; footprint NixieClockMaster:C025-024X044 -> NixieClockMaster:C_Radial_D6.3_L11.2_P2.5
- Q2, Q3: value BSS138 -> 2N7000; footprint NixieClockMaster:SOT-23_Handsoldering -> Package_TO_SOT_THT:TO-92_Inline
- R10, R11, R12, R13: footprint NixieClockMaster:R_1206_HandSoldering -> NixieClockMaster:R-0207_2V
- U1: value AP111733 -> WeMos_mini; footprint NixieClockMaster:SOT-223 -> NixieClockMaster:WeMos_D1_mini_board_flipped
- moved BT1 154.4 mm to (335.3, 152.7), turned to 180 degrees
- moved R13 140.7 mm to (198.4, 149.7), turned to 0 degrees
- moved Q2 140.5 mm to (202.2, 161.2), turned to 180 degrees
- moved Q3 140.0 mm to (202.2, 152.9), turned to 180 degrees
- moved R11 137.2 mm to (198.4, 158.1), turned to 0 degrees
- moved R12 132.6 mm to (203.5, 149.7), turned to 180 degrees
- moved R10 131.9 mm to (203.4, 158.1)
- moved U1 97.1 mm to (230.8, 159.8)
- moved SV4 88.9 mm to (268.5, 162.8), turned to 180 degrees
- moved SV2 56.6 mm to (253.4, 162.8)
- moved R9 40.1 mm to (253.2, 157.9), turned to 180 degrees
- moved C21 28.1 mm to (310.8, 151.5)
- moved U5 28.1 mm to (313.6, 155.3)
- moved Y1 28.1 mm to (314.1, 157.7)
- moved R7 21.7 mm to (192.8, 158.0), turned to 180 degrees
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- renumbered Q4 to Q6, 2N3906 to Q7
Connections:
- C7 pad 1: GND -> /VCC
- C7 pad 2: /XTAL1 -> GND
- C8 pad 1: /XTAL2 -> /VCC
- LED6 pad 4: /DATA0 -> /LED_DATA
- Q2 pad 1: /3V3 -> /DATA1_3V3
- Q2 pad 2: Net-(P1-Pad5) -> /3V3
- Q2 pad 3: /SDA -> /DATA1
- Q3 pad 1: /3V3 -> /BLANK_3V3
- Q3 pad 2: Net-(P1-Pad3) -> /3V3
- Q3 pad 3: /SCL -> /BLANK
- R10 pad 1: /SDA -> /3V3
- R10 pad 2: /VCC -> /DATA1_3V3
- R11 pad 1: /SCL -> /VCC
- R11 pad 2: /VCC -> /DATA1
- R12 pad 2: Net-(P1-Pad5) -> /BLANK_3V3
- R13 pad 1: /3V3 -> /VCC
- R13 pad 2: Net-(P1-Pad3) -> /BLANK
- R7 pad 1: /RESET -> /3V3
- R7 pad 2: /VCC -> /CLK_3V3
- U1 pad 1: GND -> /VCC
- U1 pad 2: /3V3 -> GND
- U1 pad 3: /VCC -> /PIR
- U1 pad 4: (no net) -> /BTN1
- U3 pad 27: /DATA1 -> /DATA2
- U4 pad 18: Net-(U4-Pad18) -> /DATA2
- U4 pad 27: /DATA2 -> /DATA1
Routing:
- net /DATA0: track 174.7 -> 0.00 mm, vias 1 -> 0
- net /LED_DATA: track 0.00 -> 174.4 mm
- net /SDA: track 215.6 -> 108.0 mm
- net /SCL: track 207.1 -> 106.9 mm
- net Net-(BT1-Pad1): track 118.8 -> 27.5 mm, vias 3 -> 0
- net GND: track 147.8 -> 56.6 mm, vias 5 -> 3
- net /MOSI: track 50.3 -> 0.00 mm, vias 2 -> 0
- net /RESET: track 46.3 -> 0.00 mm
- net /BLANK: track 171.7 -> 130.2 mm, vias 4 -> 3
- net /DATA2: track 68.3 -> 97.9 mm, vias 1 -> 0
- net /MISO: track 26.2 -> 0.00 mm
- net Net-(P1-Pad5): track 25.5 -> 0.00 mm, vias 1 -> 0
- net Net-(P1-Pad3): track 24.8 -> 0.00 mm, vias 1 -> 0
- net /SCK: track 24.6 -> 0.00 mm
- net /CLK_3V3: track 0.00 -> 23.2 mm
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Other:
- board size 280 x 62 mm -> 280 x 60 mm

Commit message: Improve VCC and HV layout
Parts:
- Q2, Q3, Q4, Q5: footprint Package_TO_SOT_THT:TO-92_Inline -> NixieClockMaster:TO-92_inline_2N7000
- R1, R18, R19, R2, R20, R21, R3, R4, R5, R6: footprint NixieClockMaster:R-0207_2V -> NixieClockMaster:R_Short_P7.62mm_Horizontal
- moved R5 35.4 mm to (120.8, 126.0), turned to 90 degrees
- moved R3 35.4 mm to (222.8, 126.0), turned to 90 degrees
- moved R1 17.8 mm to (321.7, 126.0), turned to 90 degrees
- moved R6 17.7 mm to (118.2, 126.0), turned to 90 degrees
- moved R2 17.6 mm to (318.7, 126.0), turned to 90 degrees
- moved R4 17.0 mm to (219.1, 126.0), turned to 90 degrees
- moved J1 15.7 mm to (353.5, 140.7), turned to 0 degrees
- moved LED7 13.7 mm to (351.9, 153.2)
- moved R19 12.4 mm to (263.3, 118.2), turned to 270 degrees
- moved R21 12.4 mm to (178.0, 118.4), turned to 270 degrees
- moved R8 12.2 mm to (351.9, 149.3)
- moved R20 8.37 mm to (163.5, 118.4), turned to 270 degrees
- moved R18 8.16 mm to (278.4, 118.0), turned to 270 degrees
- moved Q6 2.00 mm to (141.5, 158.0)
Routing:
- net /VCC: track 663.3 -> 758.5 mm, vias 12 -> 10
- net /HV: track 332.4 -> 360.6 mm
- net /LED_DATA: track 174.4 -> 158.2 mm
- net Net-(H10-PadA): track 11.0 -> 23.0 mm
- net Net-(H1-PadA): track 11.7 -> 23.3 mm
- net Net-(R6-Pad2): track 11.2 -> 22.1 mm
- net Net-(M1-PadA): track 13.7 -> 22.6 mm
- net /H1_5: track 79.4 -> 88.0 mm, vias 0 -> 1
- net Net-(R5-Pad2): track 14.4 -> 23.0 mm
- net Net-(D8-Pad2): track 17.6 -> 10.4 mm
- net /H1_9: track 70.0 -> 76.6 mm
- net GND: track 56.6 -> 50.1 mm, vias 3 -> 1
- net Net-(M10-PadA): track 15.6 -> 21.9 mm
- net Net-(D5-Pad2): track 7.14 -> 12.3 mm
- net /H1_4: track 71.8 -> 76.4 mm
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
Commit message: More minor improvements
Parts:
- moved R9 18.8 mm to (235.5, 151.7), turned to 0 degrees
- moved W2 5.59 mm to (221.3, 112.6)
- moved W3 4.49 mm to (225.5, 112.6)
Connections:
- SV4 pad 3: /VCC -> /3V3
Routing:
- net /3V3: track 64.2 -> 126.9 mm, vias 0 -> 1
- net /VCC: track 758.5 -> 763.5 mm
- net /HV: track 360.6 -> 358.2 mm
- net /DLS: track 58.0 -> 60.3 mm
- net /PIR: track 24.7 -> 26.3 mm
- net /BTN1: track 28.4 -> 29.9 mm
- net /SDA: track 107.6 -> 106.4 mm
- net /SCL: track 106.5 -> 105.9 mm
Other:
- board text added: ""Prism" IN-18 Nixie Clock"
- board text added: "3V CR1220"
- board text added: "5V PIR BTN DLS GND"
- board text added: "GND 3V3 SCL SDA"
- board text added: "HV GND VIN 5V"
- board text added: "Prototype v0.1 25/11/2018"
- board text added: "Test points"

Commit message: "Balance" HV chips
Parts:
- moved U4 15.0 mm to (174.6, 144.8)
Routing:
- net /LATCH: track 143.3 -> 112.8 mm
- net /S10_5: track 49.3 -> 72.4 mm
- net /S1_7: track 85.3 -> 106.2 mm
- net /S1_2: track 67.7 -> 88.3 mm
- net /S1_6: track 95.2 -> 115.0 mm
- net /S1_3: track 82.7 -> 101.8 mm
- net /DATA2: track 98.6 -> 80.2 mm
- net /BLANK: track 128.9 -> 110.7 mm, vias 3 -> 2
- net /S1_1: track 62.4 -> 80.5 mm
- net /S10_6: track 58.6 -> 76.4 mm
- net /S10_7: track 65.1 -> 81.5 mm
- net /S1_8: track 69.6 -> 85.9 mm
- net /S1_9: track 52.7 -> 68.9 mm
- net /S1_4: track 69.1 -> 85.0 mm
- net /S1_5: track 70.7 -> 86.0 mm
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