File: PrismDDIN18.kicad_pcb (KiCad board)
At the start: 2 copper layers, 280 x 60 mm, 76 parts, among them CON1 BARREL_JACK, IC1 LM2596T-5, J1 LED_TEST, J2 EXT_LED_OUT, M1 Z566M, M10 Z566M, SW1 SW_Push, U1 WeMos_mini, U2 HVSMPS-34063, U3 HV5622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

Commit message: Rotate tubes
Parts:
- H1, H10, M1, M10, S1, S10: value Z566M -> IN-18
- turned H1 to 356 degrees
- turned H10 to 356 degrees
- turned M1 to 356 degrees
- turned M10 to 356 degrees
- turned S1 to 356 degrees
- turned S10 to 356 degrees

Commit message: Change pin size of socket, swap D0 and D5 for PWM blanking
Parts:
- H1, H10, M1, M10, S1, S10: value IN-18 -> Z566M; footprint NixieClockMaster:IN-18-standoff-pins -> NixieClockMaster:IN-18-standoff-pins-1mm
Connections:
- U1 pad 11: /BLANK_3V3 -> /LATCH_3V3
- U1 pad 12: /LATCH_3V3 -> /BLANK_3V3
- U1 pad 15: (no net) -> Net-(U1-Pad15)
- U1 pad 8: (no net) -> Net-(U1-Pad8)
- U1 pad 9: (no net) -> Net-(U1-Pad9)
- U3 pad 18: (no net) -> Net-(U3-Pad18)
- U5 pad 7: (no net) -> Net-(U5-Pad7)
Routing:
- net /VCC: track 662.9 -> 598.3 mm
- net /S10_9: track 43.5 -> 41.2 mm
- net /H1_9: track 77.4 -> 75.4 mm
- net /BLANK_3V3: track 21.0 -> 19.3 mm
- net /H1_4: track 75.3 -> 73.7 mm
- net /LATCH_3V3: track 7.06 -> 7.96 mm
- net /S10_8: track 60.9 -> 61.8 mm
- net /M10_8: track 36.3 -> 37.2 mm
- net /S1_8: track 85.3 -> 86.2 mm
- net /H1_0: track 65.5 -> 64.6 mm
- net /S10_7: track 81.9 -> 82.8 mm
- net /M1_0: track 40.2 -> 39.3 mm
- net /S1_2: track 87.1 -> 87.9 mm
- net /S10_2: track 64.7 -> 65.5 mm
- net /M1_9: track 41.7 -> 40.9 mm
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
Commit message: Prepare for FAB
Routing:
- net /M1_4: track 57.9 -> 55.1 mm
- net /H10_4: track 106.0 -> 103.6 mm
- net /M1_5: track 61.6 -> 63.6 mm
- net /H1_6: track 61.9 -> 63.4 mm
- net /S10_6: track 88.6 -> 90.0 mm
- net /M10_6: track 64.4 -> 65.7 mm
- net /S10_7: track 82.8 -> 81.5 mm
- net /PWR_VIN: track 455.1 -> 456.2 mm
- net /H10_6: track 89.3 -> 90.3 mm
- net /M1_6: track 42.0 -> 42.9 mm
- net /S10_3: track 73.8 -> 73.0 mm
- net Net-(M10-PadA): track 20.6 -> 21.3 mm
- net Net-(LED2-Pad4): track 60.7 -> 61.4 mm
- net /S1_6: track 114.1 -> 114.8 mm
- net Net-(M1-PadA): track 22.4 -> 21.8 mm
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